File: pcb-mx-rgb/su120.kicad_pcb (KiCad board)
At the start: 2 copper layers, 98.8 x 98 mm, 371 parts, among them J1 MJ-4PP-9, J2 Conn_01x03, J3 Conn_01x08, J4 Conn_01x08, J5 Conn_01x03, J6 MJ-4PP-9, J7 Conn_02x05_Odd_Even, J8 Conn_02x05_Odd_Even, SW1 SW_PUSH_LED, SW10 SW_Push, SW11 SW_PUSH_LED, SW12 SW_PUSH_LED, SW13 SW_Push, SW14 SW_Push, SW15 SW_Push, SW16 SW_PUSH_LED, SW17 SW_Push, SW18 SW_Push, SW19 Rotary_Encoder_Switch, SW2 SW_PUSH_LED, SW20 Rotary_Encoder_Switch, SW21 SW_Push, SW3 SW_Push, SW4 SW_Push, SW5 SW_Push, SW6 SW_PUSH_LED, SW7 SW_PUSH_LED, SW8 SW_Push, SW9 SW_Push, U1 ProMicro

Commit message: Mostly done.
- Completed cleanup and conversion of schematics
- Added 100n capacitors to each LED chip
- Re-routed most of the PCB
- Moved 2u key around to adopt a column-based approach and have 4 columns of 4 keys each per PCB
- Fixed almost all DRC error, including board outline not closed
- Note: VCC (for LEDs) is routed per column but NOT supplied from USB!
Parts:
- removed the ? at (39.3, 150.4)
- removed the ? at (120.7, 116.7)
- removed the ? at (47.2, 150.4)
- removed the ? at (134.9, 116.7)
- removed the ? at (47.2, 142.1)
- removed the ? at (73.0, 135.7)
- removed the ? at (87.3, 135.7)
- removed the ? at (120.7, 135.7)
- removed the ? at (134.9, 135.7)
- removed the ? at (134.9, 150.0)
- removed the ? at (47.2, 145.7)
- removed the ? at (120.7, 150.0)
- removed the ? at (87.3, 150.0)
- removed the ? at (73.0, 150.0)
- removed the ? at (43.3, 142.1)
- removed the ? at (43.3, 135.3)
- removed the ? at (47.2, 135.3)
- removed the ? at (51.2, 142.1)
- removed the ? at (43.3, 150.4)
- removed the ? at (43.3, 145.7)
- removed the ? at (61.1, 152.4)
- removed the ? at (118.3, 152.4)
- removed the ? at (51.2, 145.7)
- removed the ? at (137.3, 152.4)
- removed the ? at (137.3, 133.3)
- removed the ? at (137.3, 114.3)
- removed the ? at (99.2, 133.4)
- removed the ? at (118.3, 133.4)
- removed the ? at (118.3, 114.3)
- removed the ? at (51.2, 135.3)
- removed the ? at (118.3, 95.3)
- removed the ? at (90.5, 143.3)
- removed the ? at (127.8, 142.9)
- removed the ? at (51.2, 150.4)
- removed the ? at (80.2, 142.9)
- removed the ? at (127.8, 123.8)
- removed the ? at (127.8, 104.8)
- removed the ? at (55.2, 142.1)
- removed the ? at (70.2, 143.3)
- removed the ? at (55.2, 145.7)
- removed the ? at (55.2, 135.3)
- removed the ? at (55.2, 150.4)
- removed the ? at (59.1, 135.4)
- removed the ? at (59.1, 150.4)
- removed the ? at (39.3, 142.5)
- removed the ? at (39.3, 135.3)
- removed the ? at (59.1, 141.8)
- removed the ? at (39.3, 145.7)
- removed the ? at (134.9, 111.9)
- removed the ? at (120.7, 111.9)
- removed H156: MountingHole_Pad, #footprint:1pin_conn
- removed the SW10 at (127.8, 104.8)
- removed the SW14 at (108.7, 123.8)
- removed the SW17 at (108.7, 142.9)
- removed the SW21 at (127.8, 142.9)
- added ?: , #footprint:M1.4_tapping_Hole_rev2, F.Cu at (40.1, 145.7)
- added ?: , #footprint:M1.4_tapping_Hole_rev2, F.Cu at (40.1, 150.4)
- added ?: , #footprint:M1.4_tapping_Hole_rev2, F.Cu at (77.8, 135.7)
- added ?: , #footprint:M1.4_tapping_Hole_rev2, F.Cu at (77.8, 150.0)
- added ?: , #footprint:M1.4_tapping_Hole_rev2, F.Cu at (124.2, 150.4)
- added ?: , #footprint:M1.4_tapping_Hole_rev2, F.Cu at (120.7, 121.4)
- added ?: , #footprint:M1.4_tapping_Hole_rev2, F.Cu at (120.7, 107.2)
- added ?: , #footprint:M1.4_tapping_Hole_rev2, F.Cu at (82.5, 135.7)
- added ?: , #footprint:M1.4_tapping_Hole_rev2, F.Cu at (124.2, 142.1)
- added ?: , #footprint:M1.4_tapping_Hole_rev2, F.Cu at (82.5, 150.0)
- added ?: , #footprint:M1.4_tapping_Hole_rev2, F.Cu at (134.9, 107.2)
- added ?: , #footprint:M1.4_tapping_Hole_rev2, F.Cu at (134.9, 121.4)
- added ?: , #footprint:M1.4_tapping_Hole_rev2, F.Cu at (120.3, 142.1)
- added ?: , #footprint:M1.4_tapping_Hole_rev2, F.Cu at (120.3, 135.3)
- added ?: , #footprint:M1.4_tapping_Hole_rev2, F.Cu at (124.2, 145.7)
- added ?: , #footprint:M1.4_tapping_Hole_rev2, F.Cu at (124.2, 135.3)
- added ?: , #footprint:M1.4_tapping_Hole_rev2, F.Cu at (120.3, 150.4)
- added ?: , #footprint:M1.4_tapping_Hole_rev2, F.Cu at (120.3, 145.7)
- added ?: , #footprint:M2_Hole, F.Cu at (99.2, 133.3)
- added ?: , #footprint:M1.4_tapping_Hole_rev2, F.Cu at (128.2, 142.1)
- added ?: , #footprint:M2_Hole, F.Cu at (80.2, 133.3)
- added ?: , #footprint:M2_Hole, F.Cu at (118.3, 95.3)
- added ?: , #footprint:M2_Hole, F.Cu at (80.2, 152.4)
- added ?: , #footprint:M2_Hole, F.Cu at (61.1, 152.4)
- added ?: , #footprint:M1.4_tapping_Hole_rev2, F.Cu at (128.2, 145.7)
- added ?: , #footprint:CherryMX_MidHeight_Choc_Silk_Line, F.Cu at (128.2, 104.0)
- added ?: , #footprint:CherryMX_MidHeight_Choc_Silk, F.Cu at (89.7, 142.9)
- added ?: , #footprint:CherryMX_MidHeight_Choc_Silk, F.Cu at (127.8, 114.3)
- added ?: , #footprint:M1.4_tapping_Hole_rev2, F.Cu at (128.2, 135.3)
- added ?: , #footprint:CherryMX_MidHeight_Choc_Silk, F.Cu at (70.6, 142.9)
- added ?: , #footprint:CherryMX_MidHeight_Choc_Silk, F.Cu at (51.6, 142.9)
- added ?: , #footprint:M1.4_tapping_Hole_rev2, F.Cu at (128.2, 150.4)
- added ?: , #footprint:CherryMX_MidHeight_Choc_Silk_Line, F.Cu at (128.2, 124.2)
- added ?: , #footprint:M1.4_tapping_Hole_rev2, F.Cu at (132.2, 142.1)
- added ?: , #footprint:M1.4_tapping_Hole_rev2, F.Cu at (132.2, 145.7)
- added ?: , #footprint:M1.4_tapping_Hole_rev2, F.Cu at (132.2, 135.3)
- added ?: , #footprint:M1.4_tapping_Hole_rev2, F.Cu at (132.2, 150.4)
- added ?: , #footprint:M1.4_tapping_Hole_rev2, F.Cu at (136.1, 135.4)
- added ?: , #footprint:M1.4_tapping_Hole_rev2, F.Cu at (136.1, 150.4)
- added ?: , #footprint:M1.4_tapping_Hole_rev2, F.Cu at (40.1, 142.5)
- added ?: , #footprint:M1.4_tapping_Hole_rev2, F.Cu at (40.1, 135.3)
- added ?: , #footprint:M1.4_tapping_Hole_rev2, F.Cu at (136.1, 141.8)
- added ?: , #footprint:M1.4_tapping_Hole_rev2, F.Cu at (44.5, 135.7)
- added ?: , #footprint:M1.4_tapping_Hole_rev2, F.Cu at (58.7, 135.7)
- added ?: , #footprint:M1.4_tapping_Hole_rev2, F.Cu at (58.7, 150.0)
- added ?: , #footprint:M1.4_tapping_Hole_rev2, F.Cu at (44.5, 150.0)
- added C1: 100n, Capacitor_SMD:C_0603_1608Metric_Pad1.08x0.95mm_HandSolder, B.Cu at (51.6, 93.5)
- added C10: 100n, Capacitor_SMD:C_0603_1608Metric_Pad1.08x0.95mm_HandSolder, B.Cu at (89.7, 112.6)
- added C11: 100n, Capacitor_SMD:C_0603_1608Metric_Pad1.08x0.95mm_HandSolder, B.Cu at (89.7, 131.6)
- added C12: 100n, Capacitor_SMD:C_0603_1608Metric_Pad1.08x0.95mm_HandSolder, B.Cu at (89.7, 150.7)
- added C13: 100n, Capacitor_SMD:C_0603_1608Metric_Pad1.08x0.95mm_HandSolder, B.Cu at (108.7, 93.5)
- added C14: 100n, Capacitor_SMD:C_0603_1608Metric_Pad1.08x0.95mm_HandSolder, B.Cu at (108.7, 112.6)
- added C15: 100n, Capacitor_SMD:C_0603_1608Metric_Pad1.08x0.95mm_HandSolder, B.Cu at (108.7, 131.6)
- added C16: 100n, Capacitor_SMD:C_0603_1608Metric_Pad1.08x0.95mm_HandSolder, B.Cu at (108.7, 150.7)
- added C17: 100n, Capacitor_SMD:C_0603_1608Metric_Pad1.08x0.95mm_HandSolder, B.Cu at (127.8, 93.5)
- added C18: 100n, Capacitor_SMD:C_0603_1608Metric_Pad1.08x0.95mm_HandSolder, B.Cu at (135.6, 114.3)
- added C2: 100n, Capacitor_SMD:C_0603_1608Metric_Pad1.08x0.95mm_HandSolder, B.Cu at (51.6, 112.6)
- added C3: 100n, Capacitor_SMD:C_0603_1608Metric_Pad1.08x0.95mm_HandSolder, B.Cu at (51.6, 131.6)
- added C4: 100n, Capacitor_SMD:C_0603_1608Metric_Pad1.08x0.95mm_HandSolder, B.Cu at (51.6, 150.7)
- added C5: 100n, Capacitor_SMD:C_0603_1608Metric_Pad1.08x0.95mm_HandSolder, B.Cu at (70.6, 93.5)
- added C6: 100n, Capacitor_SMD:C_0603_1608Metric_Pad1.08x0.95mm_HandSolder, B.Cu at (70.6, 112.6)
- added C7: 100n, Capacitor_SMD:C_0603_1608Metric_Pad1.08x0.95mm_HandSolder, B.Cu at (70.6, 131.6)
- added C8: 100n, Capacitor_SMD:C_0603_1608Metric_Pad1.08x0.95mm_HandSolder, B.Cu at (70.6, 150.7)
- added C9: 100n, Capacitor_SMD:C_0603_1608Metric_Pad1.08x0.95mm_HandSolder, B.Cu at (89.7, 93.5)
- added H100: MountingHole_Pad, #footprint:1pin_conn, F.Cu at (116.6, 89.7)
- added H101: MountingHole_Pad, #footprint:1pin_conn, F.Cu at (112.7, 93.5)
- added H102: MountingHole_Pad, #footprint:1pin_conn, F.Cu at (116.6, 108.8)
- added H103: MountingHole_Pad, #footprint:1pin_conn, F.Cu at (112.7, 112.6)
- added H104: MountingHole_Pad, #footprint:1pin_conn, F.Cu at (116.6, 127.8)
- added H105: MountingHole_Pad, #footprint:1pin_conn, F.Cu at (112.7, 131.6)
- added H106: MountingHole_Pad, #footprint:1pin_conn, F.Cu at (116.6, 146.9)
- added H107: MountingHole_Pad, #footprint:1pin_conn, F.Cu at (112.7, 150.7)
- added H110: MountingHole_Pad, #footprint:1pin_conn, F.Cu at (43.8, 146.9)
- added H111: MountingHole_Pad, #footprint:1pin_conn, F.Cu at (59.4, 140.0)
- added H112: MountingHole_Pad, #footprint:1pin_conn, F.Cu at (62.8, 146.9)
- added H141: MountingHole_Pad, #footprint:1pin_conn, F.Cu at (78.5, 140.0)
- added H142: MountingHole_Pad, #footprint:1pin_conn, F.Cu at (81.9, 146.9)
- added H143: MountingHole_Pad, #footprint:1pin_conn, F.Cu at (97.5, 140.0)
- added H144: MountingHole_Pad, #footprint:1pin_conn, F.Cu at (131.8, 93.5)
- added H145: MountingHole_Pad, #footprint:1pin_conn, F.Cu at (135.6, 89.7)
- added H146: MountingHole_Pad, #footprint:1pin_conn, F.Cu at (55.6, 150.7)
- added H147: MountingHole_Pad, #footprint:1pin_conn, F.Cu at (59.4, 146.9)
- added H148: MountingHole_Pad, #footprint:1pin_conn, F.Cu at (74.6, 150.7)
- added H149: MountingHole_Pad, #footprint:1pin_conn, F.Cu at (78.5, 146.9)
- added H150: MountingHole_Pad, #footprint:1pin_conn, F.Cu at (93.7, 150.7)
- added H151: MountingHole_Pad, #footprint:1pin_conn, F.Cu at (97.5, 146.9)
- added H59: MountingHole_Pad, #footprint:1pin_conn, F.Cu at (59.4, 89.7)
- added H60: MountingHole_Pad, #footprint:1pin_conn, F.Cu at (55.6, 112.6)
- added H79: MountingHole_Pad, #footprint:1pin_conn, F.Cu at (135.6, 110.3)
- added H80: MountingHole_Pad, #footprint:1pin_conn, F.Cu at (81.9, 89.7)
- added H81: MountingHole_Pad, #footprint:1pin_conn, F.Cu at (97.5, 82.9)
- added H82: MountingHole_Pad, #footprint:1pin_conn, F.Cu at (81.9, 108.8)
- added H83: MountingHole_Pad, #footprint:1pin_conn, F.Cu at (97.5, 101.9)
- added H84: MountingHole_Pad, #footprint:1pin_conn, F.Cu at (81.9, 127.8)
- added H85: MountingHole_Pad, #footprint:1pin_conn, F.Cu at (97.5, 121.0)
- added H86: MountingHole_Pad, #footprint:1pin_conn, F.Cu at (93.7, 93.5)
- added H87: MountingHole_Pad, #footprint:1pin_conn, F.Cu at (97.5, 89.7)
- added H88: MountingHole_Pad, #footprint:1pin_conn, F.Cu at (93.7, 112.6)
- added H89: MountingHole_Pad, #footprint:1pin_conn, F.Cu at (97.5, 108.8)
- added H90: MountingHole_Pad, #footprint:1pin_conn, F.Cu at (93.7, 131.6)
- added H91: MountingHole_Pad, #footprint:1pin_conn, F.Cu at (97.5, 127.8)
- added H92: MountingHole_Pad, #footprint:1pin_conn, F.Cu at (116.6, 82.9)
- added H93: MountingHole_Pad, #footprint:1pin_conn, F.Cu at (100.9, 89.7)
- added H94: MountingHole_Pad, #footprint:1pin_conn, F.Cu at (116.4, 102.1)
- added H95: MountingHole_Pad, #footprint:1pin_conn, F.Cu at (100.9, 108.8)
- added H96: MountingHole_Pad, #footprint:1pin_conn, F.Cu at (116.6, 121.0)
- added H97: MountingHole_Pad, #footprint:1pin_conn, F.Cu at (100.9, 127.8)
- added H98: MountingHole_Pad, #footprint:1pin_conn, F.Cu at (116.6, 140.0)
- added H99: MountingHole_Pad, #footprint:1pin_conn, F.Cu at (100.9, 146.9)
- added SW12: SW_PUSH_LED, #footprint:CherryMX_MidHeight_RGB_Hotswap, F.Cu at (89.7, 142.9)
- added SW18: SW_PUSH_LED, #footprint:CherryMX_MidHeight_RGB_Hotswap, F.Cu at (127.8, 114.3)
- added SW4: SW_PUSH_LED, #footprint:CherryMX_MidHeight_RGB_Hotswap, F.Cu at (51.6, 142.9)
- added SW8: SW_PUSH_LED, #footprint:CherryMX_MidHeight_RGB_Hotswap, F.Cu at (70.6, 142.9)
- SW10: renamed from SW8; value SW_Push -> SW_PUSH_LED; footprint #footprint:CherryMX_MidHeight_Choc_Hotswap_rev5 -> #footprint:CherryMX_MidHeight_RGB_Hotswap
- SW11: renamed from SW13; value SW_Push -> SW_PUSH_LED; footprint #footprint:CherryMX_MidHeight_Choc_Hotswap_rev5 -> #footprint:CherryMX_MidHeight_RGB_Hotswap
- SW13: renamed from SW4; value SW_Push -> SW_PUSH_LED; footprint #footprint:CherryMX_MidHeight_Choc_Hotswap_rev5 -> #footprint:CherryMX_MidHeight_RGB_Hotswap
- SW14: renamed from SW9; value SW_Push -> SW_PUSH_LED; footprint #footprint:CherryMX_MidHeight_Choc_Hotswap_rev5 -> #footprint:CherryMX_MidHeight_RGB_Hotswap
- SW15: value SW_Push -> SW_PUSH_LED; footprint #footprint:CherryMX_MidHeight_Choc_Hotswap_rev5 -> #footprint:CherryMX_MidHeight_RGB_Hotswap
- SW17: renamed from SW5; value SW_Push -> SW_PUSH_LED; footprint #footprint:CherryMX_MidHeight_Choc_Hotswap_rev5 -> #footprint:CherryMX_MidHeight_RGB_Hotswap
- SW9: renamed from SW3; value SW_Push -> SW_PUSH_LED; footprint #footprint:CherryMX_MidHeight_Choc_Hotswap_rev5 -> #footprint:CherryMX_MidHeight_RGB_Hotswap
- moved H71 106.8 mm to (131.8, 122.1)
- moved H78 104.9 mm to (131.8, 106.5)
- moved H70 93.9 mm to (124.9, 106.5)
- moved H109 85.5 mm to (135.6, 82.9), turned to 0 degrees
- moved H40 85.3 mm to (59.4, 143.3)
- moved H25 85.3 mm to (47.2, 135.1)
- moved D10 85.3 mm to (49.6, 135.1)
- moved H39 85.1 mm to (43.8, 143.3)
- moved H30 84.8 mm to (47.6, 150.7)
- moved H43 68.1 mm to (135.6, 118.3), turned to 90 degrees
- moved H49 66.5 mm to (128.2, 131.8), turned to 90 degrees
- moved H76 65.5 mm to (78.5, 127.8)
- moved H77 64.9 mm to (74.6, 131.6)
- moved H108 60.5 mm to (120.0, 89.7), turned to 0 degrees
- moved H132 60.4 mm to (78.5, 143.3)
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- renumbered H101 to H51, H102 to H52, H103 to H53, H104 to H54, H105 to H55, H106 to H56, H107 to H58, H110 to H61, H111 to H62, H112 to H63, H141 to H64, H142 to H65, H143 to H66, H144 to H67, H145 to H68, H146 to H69, H147 to H70, H148 to H71, H149 to H72, H150 to H73, H151 to H74, H152 to H75, H153 to H76, H154 to H77, H155 to H78, SW6 to SW2, SW19 to SW20, SW20 to SW21, SW18 to SW22, SW11 to SW3, SW2 to SW5, SW7 to SW6, SW12 to SW7
Connections:
- D10 pad 1: Y2 -> Y4
- D15 pad 1: Y3 -> Y4
- D16 pad 1: Y4 -> Y2
- H108 pad 1: Net-(H103-Pad1) -> Net-(H100-Pad1)
- H109 pad 1: VCC -> GND
- H117 pad 1: X5 -> X2
- H122 pad 1: X5 -> X2
- H131 pad 1: Y3 -> Y4
- H132 pad 1: Y3 -> Y4
- H210 pad 1: X5 -> X3
- H211 pad 1: X5 -> X3
- H25 pad 1: X5 -> X1
- H30 pad 1: X5 -> X1
- H39 pad 1: Y2 -> Y4
- H40 pad 1: Y2 -> Y4
- H41 pad 1: X2 -> X5
- H43 pad 1: X2 -> X5
- H45 pad 1: Y4 -> Y2
- H46 pad 1: Y4 -> Y2
- H49 pad 1: Y4 -> Y2
- H50 pad 1: Y4 -> Y2
- H53 pad 1: Net-(H103-Pad1) -> Net-(H53-Pad1)
- H63 pad 1: Net-(H112-Pad1) -> Net-(H110-Pad1)
- H69 pad 1: Net-(H146-Pad1) -> Net-(H149-Pad1)
- H71 pad 1: Net-(H112-Pad1) -> Net-(H145-Pad1)
- H72 pad 1: Net-(H149-Pad1) -> Net-(H72-Pad1)
- H78 pad 1: Net-(H146-Pad1) -> Net-(H78-Pad1)
- SW1 pad 2: Net-(H103-Pad1) -> Net-(H53-Pad1)
- SW10 pad 1: X3 -> VCC
- SW10 pad 2: Net-(D8-Pad2) -> Net-(H84-Pad1)
- SW11 pad 1: X3 -> VCC
- SW11 pad 2: Net-(D13-Pad2) -> Net-(H142-Pad1)
- SW13 pad 1: X4 -> VCC
- SW13 pad 2: Net-(D4-Pad2) -> Net-(H100-Pad1)
- SW14 pad 1: X4 -> VCC
- SW14 pad 2: Net-(D9-Pad2) -> Net-(H102-Pad1)
- SW15 pad 1: X5 -> VCC
- SW15 pad 2: Net-(D15-Pad2) -> Net-(H104-Pad1)
- SW16 pad 2: Net-(H146-Pad1) -> Net-(H106-Pad1)
- SW16 pad 4: Net-(H112-Pad1) -> Net-(H151-Pad1)
- SW16 pad 5: X2 -> X4
- SW16 pad 6: Net-(D16-Pad2) -> Net-(D17-Pad2)
- SW17 pad 1: X5 -> VCC
- SW17 pad 2: Net-(D5-Pad2) -> Net-(H145-Pad1)
- SW2 pad 4: Net-(H103-Pad1) -> Net-(H53-Pad1)
- SW3 pad 2: Net-(H112-Pad1) -> Net-(H110-Pad1)
- SW5 pad 2: Net-(H149-Pad1) -> Net-(H72-Pad1)
- SW7 pad 4: Net-(H146-Pad1) -> Net-(H149-Pad1)
- SW9 pad 1: X3 -> VCC
- SW9 pad 2: Net-(D3-Pad2) -> Net-(H82-Pad1)
Routing:
- net GND: track 1083.6 -> 358.9 mm, vias 129 -> 250
- net VCC: track 97.3 -> 452.5 mm
- net Y3: track 311.7 -> 248.6 mm, vias 6 -> 2
- net Net-(H145-Pad1): track 0.00 -> 56.9 mm, vias 0 -> 3
- net Y2: track 265.5 -> 312.8 mm, vias 2 -> 1
- net Net-(H103-Pad1): track 43.9 -> 0.00 mm, vias 2 -> 0
- net Net-(H82-Pad1): track 0.00 -> 43.2 mm, vias 0 -> 2
- net Net-(H84-Pad1): track 0.00 -> 43.1 mm, vias 0 -> 2
- net Net-(H53-Pad1): track 0.00 -> 43.1 mm, vias 0 -> 2
- net Net-(H110-Pad1): track 0.00 -> 43.0 mm, vias 0 -> 2
- net Net-(H142-Pad1): track 0.00 -> 42.9 mm, vias 0 -> 2
- net Net-(H55-Pad1): track 5.21 -> 43.0 mm, vias 0 -> 2
- net Net-(H102-Pad1): track 0.00 -> 37.5 mm, vias 0 -> 2
- net Net-(H149-Pad1): track 0.00 -> 37.3 mm, vias 0 -> 2
- net Net-(H67-Pad1): track 0.00 -> 37.1 mm, vias 0 -> 2
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Other:
- outline, holes or cut-outs redrawn
- net class Small added: clearance 0.1524, trace_width 0.1524, via_dia 0.8, via_drill 0.4
- rule trace_min: 0.2 -> 0.1524
- board text added: "DIN"
- board text added: "DOUT"
- board text added: "SU120 "YAKITORI" RGB Rev.1 by @AxelVoitier"
- board text removed: "SU120 "YAKITORI" Rev.8 by @e3w2q"
