File: pcb-mx-rgb/su120.sch (KiCad schematic (older format))
At the start: 167 parts, among them J1 MJ-4PP-9, J2 Conn_01x03, J3 Conn_01x08, J4 Conn_01x08, J5 Conn_01x03, J6 MJ-4PP-9, J7 Conn_02x05_Odd_Even, J8 Conn_02x05_Odd_Even, SW1 SW_PUSH_LED, SW10 SW_Push, SW11 SW_PUSH_LED, SW12 SW_PUSH_LED, SW13 SW_Push, SW14 SW_Push, SW15 SW_Push, SW16 SW_PUSH_LED, SW17 SW_Push, SW18 SW_Push, SW19 Rotary_Encoder_Switch, SW2 SW_PUSH_LED, SW20 Rotary_Encoder_Switch, SW21 SW_Push, SW3 SW_Push, SW4 SW_Push, SW5 SW_Push, SW6 SW_PUSH_LED, SW7 SW_PUSH_LED, SW8 SW_Push, SW9 SW_Push, U1 ProMicro

Commit message: Mostly done.
- Completed cleanup and conversion of schematics
- Added 100n capacitors to each LED chip
- Re-routed most of the PCB
- Moved 2u key around to adopt a column-based approach and have 4 columns of 4 keys each per PCB
- Fixed almost all DRC error, including board outline not closed
- Note: VCC (for LEDs) is routed per column but NOT supplied from USB!
Parts:
- added C1, C10, C11, C12, C13, C14, C15, C16, C17, C18, C2, C3, C4, C5, C6, C7, C8, C9: 100n, Capacitor_SMD:C_0603_1608Metric_Pad1.08x0.95mm_HandSolder, symbol Device:C_Small
- added H100, H101, H102, H103, H104, H105, H106, H107, H108, H109, H110, H111, H112, H141, H142, H143, H144, H145, H146, H147, H148, H149, H150, H151, H80, H81, H82, H83, H84, H85, H86, H87, H88, H89, H90, H91, H92, H93, H94, H95, H96, H97, H98, H99: MountingHole_Pad, #footprint:1pin_conn, symbol Connector:TestPoint
- added unit 2 of SW10
- added unit 2 of SW11
- added unit 2 of SW12
- added unit 2 of SW13
- added unit 2 of SW14
- added unit 2 of SW15
- added unit 2 of SW16
- added unit 2 of SW17
- added unit 2 of SW4
- added unit 2 of SW8
- added unit 2 of SW9
- H10, H115, H116, H117, H120, H121, H122, H127, H128, H129, H130, H131, H132, H133, H134, H135, H136, H137, H138, H139, H140, H15, H16, H17, H18, H19, H20, H210, H211, H212, H213, H23, H24, H25, H28, H29, H3, H30, H35, H36, H37, H38, H39, H4, H40, H42, H44, H47, H48, H5, H8, H9: symbol Mechanical:MountingHole_Pad -> Connector:TestPoint
- SW1: footprint SofleRGB:Choc_Hotswap_SK6812MiniE -> #footprint:CherryMX_MidHeight_RGB_Hotswap
- SW10: renamed from SW8; value SW_Push -> SW_PUSH_LED; footprint #footprint:CherryMX_MidHeight_Choc_Hotswap_rev5 -> #footprint:CherryMX_MidHeight_RGB_Hotswap; symbol Switch:SW_Push -> Sofle:SW_PUSH_LED
- SW11: renamed from SW13; value SW_Push -> SW_PUSH_LED; footprint #footprint:CherryMX_MidHeight_Choc_Hotswap_rev5 -> #footprint:CherryMX_MidHeight_RGB_Hotswap; symbol Switch:SW_Push -> Sofle:SW_PUSH_LED
- SW12: renamed from SW21; value SW_Push -> SW_PUSH_LED; footprint #footprint:CherryMX_MidHeight_Choc_Hotswap_rev5 -> #footprint:CherryMX_MidHeight_RGB_Hotswap; symbol Switch:SW_Push -> Sofle:SW_PUSH_LED
- SW13: renamed from SW4; value SW_Push -> SW_PUSH_LED; footprint #footprint:CherryMX_MidHeight_Choc_Hotswap_rev5 -> #footprint:CherryMX_MidHeight_RGB_Hotswap; symbol Switch:SW_Push -> Sofle:SW_PUSH_LED
- SW14: renamed from SW9; value SW_Push -> SW_PUSH_LED; footprint #footprint:CherryMX_MidHeight_Choc_Hotswap_rev5 -> #footprint:CherryMX_MidHeight_RGB_Hotswap; symbol Switch:SW_Push -> Sofle:SW_PUSH_LED
- SW15: renamed from SW14; value SW_Push -> SW_PUSH_LED; footprint #footprint:CherryMX_MidHeight_Choc_Hotswap_rev5 -> #footprint:CherryMX_MidHeight_RGB_Hotswap; symbol Switch:SW_Push -> Sofle:SW_PUSH_LED
- SW16: renamed from SW17; value SW_Push -> SW_PUSH_LED; footprint #footprint:CherryMX_MidHeight_Choc_Hotswap_rev5 -> #footprint:CherryMX_MidHeight_RGB_Hotswap; symbol Switch:SW_Push -> Sofle:SW_PUSH_LED
- SW17: renamed from SW5; value SW_Push -> SW_PUSH_LED; footprint #footprint:CherryMX_MidHeight_Choc_Hotswap_rev5 -> #footprint:CherryMX_MidHeight_RGB_Hotswap; symbol Switch:SW_Push -> Sofle:SW_PUSH_LED
- SW18: renamed from SW16; footprint SofleRGB:Choc_Hotswap_SK6812MiniE -> #footprint:CherryMX_MidHeight_RGB_Hotswap
- SW4: renamed from SW10; value SW_Push -> SW_PUSH_LED; footprint #footprint:CherryMX_MidHeight_Choc_Hotswap_rev5 -> #footprint:CherryMX_MidHeight_RGB_Hotswap; symbol Switch:SW_Push -> Sofle:SW_PUSH_LED
- SW5: renamed from SW2; footprint SofleRGB:Choc_Hotswap_SK6812MiniE -> #footprint:CherryMX_MidHeight_RGB_Hotswap
- SW6: renamed from SW7; footprint SofleRGB:Choc_Hotswap_SK6812MiniE -> #footprint:CherryMX_MidHeight_RGB_Hotswap
- SW7: renamed from SW12; footprint SofleRGB:Choc_Hotswap_SK6812MiniE -> #footprint:CherryMX_MidHeight_RGB_Hotswap
- SW8: renamed from SW15; value SW_Push -> SW_PUSH_LED; footprint #footprint:CherryMX_MidHeight_Choc_Hotswap_rev5 -> #footprint:CherryMX_MidHeight_RGB_Hotswap; symbol Switch:SW_Push -> Sofle:SW_PUSH_LED
- SW9: renamed from SW3; value SW_Push -> SW_PUSH_LED; footprint #footprint:CherryMX_MidHeight_Choc_Hotswap_rev5 -> #footprint:CherryMX_MidHeight_RGB_Hotswap; symbol Switch:SW_Push -> Sofle:SW_PUSH_LED
- gave numbers to parts that had none: 28
- renumbered SW16 to SW18, SW6 to SW2, SW19 to SW20, SW20 to SW21, SW18 to SW22, SW11 to SW3, SW2 to SW5, SW7 to SW6, SW12 to SW7
Connections:
- net GND: now also C1.2, C10.2, C11.2, C12.2, C13.2, C14.2, C15.2, C16.2, C17.2, C18.2, C2.2, C3.2, C4.2, C5.2, C6.2, C7.2, C8.2, C9.2, H109.1, H111.1, H141.1, H143.1, H81.1, H83.1, H85.1, H92.1, H94.1, H96.1, H98.1, SW10.3 (GND), SW11.3 (GND), SW12.3 (GND), SW13.3 (GND), SW14.3 (GND), SW15.3 (GND), SW16.3 (GND), SW17.3 (GND), SW4.3 (GND), SW8.3 (GND), SW9.3 (GND)
- net VCC: now also C1.1, C10.1, C11.1, C12.1, C13.1, C14.1, C15.1, C16.1, C17.1, C18.1, C2.1, C3.1, C4.1, C5.1, C6.1, C7.1, C8.1, C9.1, H101.1, H103.1, H105.1, H107.1, H144.1, H146.1, H148.1, H150.1, H86.1, H88.1, H90.1, SW10.1 (VDD), SW11.1 (VDD), SW12.1 (VDD), SW13.1 (VDD), SW14.1 (VDD), SW15.1 (VDD), SW16.1 (VDD), SW17.1 (VDD), SW4.1 (VDD), SW8.1 (VDD), SW9.1 (VDD)
- net X1: now also H25.1, H30.1, SW4.5
- net X2: now also H117.1, H122.1, SW8.5; no longer H41.1, H43.1, SW18.5
- net X3: now also H210.1, H211.1, SW10.5, SW11.5, SW12.5, SW9.5; no longer SW10.1, SW11.1, SW9.1
- net X4: now also SW13.5, SW14.5, SW15.5, SW16.5; no longer SW13.1, SW14.1, SW15.1, SW16.1
- net X5: now also H41.1, H43.1, SW17.5, SW18.5; no longer H117.1, H122.1, H210.1, H211.1, H25.1, H30.1, SW12.1, SW17.1, SW4.1, SW8.1
- net Y2: now also D16.1 (K), H45.1, H46.1, H49.1, H50.1; no longer D10.1 (K), H39.1, H40.1
- net Y3: no longer D15.1 (K), H131.1, H132.1
- net Y4: now also D10.1 (K), D15.1 (K), H131.1, H132.1, H39.1, H40.1; no longer D16.1 (K), H45.1, H46.1, H49.1, H50.1
- net at D3.2 (A): now also SW9.6; no longer SW9.2
- net at D4.2 (A): now also SW13.6; no longer SW13.2
- net at D8.2 (A): now also SW10.6; no longer SW10.2
- net at D9.2 (A): now also SW14.6; no longer SW14.2
- net at D5.2 (A): now also SW17.6; no longer SW17.2
- net at D10.2 (A): now also SW4.6; no longer SW4.2
- net at D17.2 (A): now also SW16.6; no longer SW16.2
- net at D13.2 (A): now also SW11.6; no longer SW11.2
- net at D14.2 (A): now also SW15.6; no longer SW15.2
- net at D15.2 (A): now also SW8.6; no longer SW8.2
- net at D20.2 (A): now also SW12.6; no longer SW12.2
- net at H63.1, SW3.2 (DOUT): now also H110.1, SW4.4 (DIN); no longer H71.1, SW18.4 (DIN)
- net at H72.1, SW5.2 (DOUT): now also H80.1, SW9.4 (DIN)
- net at H69.1, SW7.4 (DIN): now also H149.1, SW8.2 (DOUT); no longer H78.1, SW18.2 (DOUT)
- new net: H78.1, SW18.2 (DOUT)
- new net: H145.1, H71.1, SW17.2 (DOUT), SW18.4 (DIN)
- new net: H84.1, H89.1, SW10.2 (DOUT), SW11.4 (DIN)
- new net: H82.1, H87.1, SW10.4 (DIN), SW9.2 (DOUT)
- new net: H142.1, H91.1, SW11.2 (DOUT), SW12.4 (DIN)
- new net: H106.1, H97.1, SW15.4 (DIN), SW16.2 (DOUT)
- new net: H151.1, H99.1, SW12.2 (DOUT), SW16.4 (DIN)
- new net: H104.1, H95.1, SW14.4 (DIN), SW15.2 (DOUT)
- new net: H102.1, H93.1, SW13.4 (DIN), SW14.2 (DOUT)
- new net: H100.1, H108.1, SW13.2 (DOUT), SW17.4 (DIN)
- new net: H112.1, H147.1, SW4.2 (DOUT), SW8.4 (DIN)
- no-connect marks 2 -> 16
Other:
- moved on the sheet: D10, D15, D16, D20, H10, H115, H116, H117, H120, H121, H122, H127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
