File: Kyfle/PCB-SU120-RGB/su120.sch (KiCad schematic (older format))
At the start: 90 parts, among them J1 MJ-4PP-9, J2 Conn_01x03, J3 Conn_01x08, J4 Conn_01x08, J6 MJ-4PP-9, SW1 SW_PUSH_LED, SW10 SW_PUSH_LED, SW11 SW_PUSH_LED, SW12 SW_PUSH_LED, SW13 SW_PUSH_LED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

Commit message: Yet another big update
- Integrated 5-way switch (instead of one of the encoder)
- Based on corrected footprint for roller encoder, it has been repositioned
- Touching up lots of silk
- 2u board made as a footprint module as well
- Fixed a potential short with 2u stabiliser metal bar on VCC and GND
- Added various 3d models
Parts:
- removed D18: D, Kyfle Footprints:diode_TH_SMD_rev3, symbol Device:D
- removed H133, H135, H136, H137, H138, H139, H170, H46, H50: MountingHole_Pad, Kyfle Footprints:1pin_rect_conn, symbol Connector:TestPoint
- removed SW19: Rotary_Encoder_Switch, Kyfle Footprints:RollerEncoder_Panasonic_EVQWGD001_No_Cutout, symbol Device:Rotary_Encoder_Switch
- removed SW20: Rotary_Encoder_Switch, Kyfle Footprints:RotaryEncoder_Alps_EC11E-Switch_Vertical_H20mm_rev2, symbol Device:Rotary_Encoder_Switch
- added H101, H102: MountingHole_Pad, Kyfle Footprints:1pin_rect_conn, symbol Connector:TestPoint
- renumbered D19 to D18, H134 to H135, H140 to H138, H171 to H170, SW23 to SW19, SW21 to SW20
Connections:
- net X10: now also D5.2 (A)
- net X4: now also H135.1, SW19.S1, SW20.S1
- net X5: now also D2.2 (A); no longer H135.1, H6.1, SW19.S1, SW20.S1, SW24.Com
- net X7: now also D1.2 (A), SW19.A, H102.1; no longer SW19.B
- net X8: now also D3.2 (A), SW19.B, H101.1; no longer SW19.A
- net X9: now also D4.2 (A)
- net Y1: no longer D1.1 (K)
- net Y2: no longer D3.1 (K)
- net Y3: no longer D4.1 (K)
- net Y4: no longer D5.1 (K)
- net Y6: now also H6.1, SW24.Com; no longer D2.1 (K)
- net at SW24.A: now also D1.1 (K); no longer D1.2 (A)
- net at SW24.B: now also D3.1 (K); no longer D3.2 (A)
- net at SW24.C: now also D4.1 (K); no longer D4.2 (A)
- net at SW24.D: now also D5.1 (K); no longer D5.2 (A)
- net at SW24.E: now also D2.1 (K); no longer D2.2 (A)
Other:
- moved on the sheet: D1, D18, D2, D3, D4, D5, H135, H138, H170, H6, SW19, SW20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
