File: Lergo/BottomPlate/LergoBottomPlate.kicad_pcb (KiCad board)
At the start: 2 copper layers, 164 x 146.3 mm, 54 parts, among them SW2 10°, SW2 15°, SW2 19°, SW2 25°, SW2 30°, SW2 35°, SW2 40°, SW2 45°, SW2 5°, SW2 KEY_SWITCH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

Commit message: Adding mounting holes in bottom plate for Keeb.io USB-C breakout board
Parts:
- added REF**: KeebIO_USB-C_Breakout, Lergo Footprints:KeebIO_USB-C_Breakout, F.Cu at (107.8, 52.1)
