File: Framework/Kicad templates/PCB/HandyWork-PCB.kicad_pcb (KiCad board)
At the start: 4 copper layers, 283.2 x 131.5 mm, 52 parts, among them J1 Conn_01x04, J2 Conn_02x04_Odd_Even, SW1 KXT3, SW2 KXT3, U1 RP2040, U2 W25Q16JV, U3 IS31FL3733B-QF, Y1 12.000 MHz

Commit message: HandyWork: Updating KiCad PCB template. Now complete.
Parts:
- added REF**: OSHW-Logo2_7.3x6mm_SilkScreen, Symbol:OSHW-Logo2_7.3x6mm_SilkScreen, B.Cu at (253.0, 143.2)
- moved J1 0.15 mm to (14.9, 144.9)
Connections:
- net /LED_CS1 renamed /LED_COL7
- net /LED_CS10 renamed /LED_COL13
- net /LED_CS11 renamed /LED_COL1
- net /LED_CS12 renamed /LED_COL3
- net /LED_CS13 renamed /LED_COL4
- net /LED_CS2 renamed /LED_COL5
- net /LED_CS3 renamed /LED_COL6
- net /LED_CS4 renamed /LED_COL8
- net /LED_CS5 renamed /LED_COL9
- net /LED_CS6 renamed /LED_COL11
- net /LED_CS7 renamed /LED_COL10
- net /LED_CS8 renamed /LED_COL12
- net /LED_CS9 renamed /LED_COL2
- net /LED_SW1 renamed /LED_ROW5
- net /LED_SW2 renamed /LED_ROW4
- net /LED_SW3 renamed /LED_ROW3
- net /LED_SW4 renamed /LED_ROW2
- net /LED_SW5 renamed /LED_ROW1
Routing:
- net /ROW5: track 0.80 -> 556.2 mm, vias 1 -> 7
- net /ROW4: track 0.80 -> 483.4 mm, vias 1 -> 3
- net /ROW3: track 0.79 -> 465.3 mm, vias 1 -> 4
- net /ROW2: track 0.79 -> 447.1 mm
- net /ROW1: track 1.19 -> 424.8 mm, vias 1 -> 2
- net /COL13: track 0.96 -> 274.7 mm, vias 1 -> 4
- net /COL12: track 1.04 -> 251.3 mm, vias 1 -> 2
- net /LED_COL13: track 0.53 -> 243.1 mm
- net /COL11: track 1.09 -> 231.3 mm, vias 1 -> 2
- net /LED_COL12: track 0.80 -> 219.7 mm
- net /COL10: track 0.72 -> 209.9 mm, vias 1 -> 2
- net /LED_COL11: track 0.89 -> 198.4 mm
- net /COL9: track 0.86 -> 189.0 mm, vias 1 -> 2
- net /LED_COL10: track 0.53 -> 177.8 mm
- net /COL8: track 0.70 -> 169.7 mm, vias 1 -> 2
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Other:
- board text added: "Designed by Axel Voitier"
- board text added: "Ergosplit keyboard for Framework Laptop 16"
- board text added: "HandyWork"
- board text added: "Licensed under CERN-OHL-W v2"
- board text added: "PCB Template"
