File: Framework/Kicad templates/PCB/HandyWork-PCB.kicad_pcb (KiCad board)
At the start: 4 copper layers, 283.2 x 131.5 mm, 53 parts, among them J1 Conn_01x04, J2 Conn_02x04_Odd_Even, SW1 KXT3, SW2 KXT3, U1 RP2040, U2 W25Q16JV, U3 IS31FL3733B-QF, Y1 12.000 MHz

Commit message: HandyWork: Refactor vias to not use 0.2mm drill in order to be significantly cheaper (~50% for the PCB itself)
Routing:
- net GND: track 44.5 -> 59.0 mm
- net /COL10: track 209.9 -> 212.5 mm
- net /SWDIO: track 9.34 -> 11.5 mm
- net /LED_COL1: track 13.0 -> 14.7 mm
- net /LED_INT: track 22.9 -> 24.5 mm
- net /COL6: track 133.4 -> 134.9 mm
- net Net-(U1-RUN): track 7.29 -> 8.78 mm
- net /COL5: track 97.3 -> 98.6 mm
- net /COL4: track 77.0 -> 78.1 mm
- net +3V3: track 23.6 -> 22.5 mm, vias 24 -> 23
- net /LED_ROW2: track 6.22 -> 5.32 mm
- net +1V1: track 20.8 -> 21.7 mm
- net /I^{2}C_SDA: track 24.4 -> 25.2 mm
- net /LED_ROW5: track 4.47 -> 3.67 mm
- net /LED_ROW3: track 5.48 -> 4.71 mm
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
Commit message: HandyWork: Fixes placement of some components around QFN packages
Fab house has a 1mm margin to apply around QFN (or QFN like) parts. Few resistors/capacitors were in that margin/courtyard.
Parts:
- moved C10 0.76 mm to (22.5, 143.4)
- moved C19 0.71 mm to (34.7, 137.0)
- moved C1 0.67 mm to (29.0, 140.5)
- moved R1 0.67 mm to (30.0, 142.4)
- moved R2 0.67 mm to (29.0, 142.4)
- moved SW1 0.45 mm to (25.6, 145.1)
- moved C20 0.39 mm to (33.5, 137.6)
- moved C14 0.27 mm to (22.5, 133.4)
- moved R12 0.10 mm to (39.0, 133.1)
- moved C5 0.08 mm to (14.1, 136.8)
Routing:
- net GND: track 59.0 -> 55.7 mm, vias 62 -> 60
- net Net-(R2-Pad1): track 2.21 -> 3.12 mm
- net Net-(U1-~{QSPI_SS}): track 8.83 -> 9.37 mm
